File: boards/temp-sensor/pcb/temp-sensor.kicad_sch (KiCad schematic)
At the start: 56 parts, among them J1 Bannana plug, J2 Bannana plug, J3 I2C, J4 UART, J5 SPI, J6 PSU, J7 CTRL, J8 Conn_02x08_Odd_Even, Q1 MMBT2222A, Q2 MMBT2222A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

Commit message: WIP Implement temp-sensor PCB
Parts:
- removed C1, C2: 100n, Capacitor_SMD:C_0603_1608Metric_Pad1.08x0.95mm_HandSolder, symbol Device:C
- removed C12: 1u, Capacitor_SMD:C_0603_1608Metric_Pad1.08x0.95mm_HandSolder, symbol Device:C
- removed D1: NCD0805R1, LED_SMD:LED_0805_2012Metric_Pad1.15x1.40mm_HandSolder, symbol Device:LED
- removed J1: Bannana plug, Connector:Banana_Cliff_FCR7350R_S16N-PC_Horizontal, symbol Connector:Conn_01x01_Socket
- removed J2: Bannana plug, Connector:Banana_Cliff_FCR7350B_S16N-PC_Horizontal, symbol Connector:Conn_01x01_Socket
- removed J5: SPI, Connector_PinHeader_2.54mm:PinHeader_1x08_P2.54mm_Vertical, symbol Connector_Generic:Conn_01x08
- removed J6: PSU, Connector_Molex:Molex_KK-254_AE-6410-04A_1x04_P2.54mm_Vertical, symbol Connector_Generic:Conn_01x04
- removed J7: CTRL, Connector_Molex:Molex_KK-254_AE-6410-04A_1x04_P2.54mm_Vertical, symbol Connector_Generic:Conn_01x04
- removed J8: Conn_02x08_Odd_Even, Connector_PinHeader_2.54mm:PinHeader_2x04_P2.54mm_Vertical, symbol Connector_Generic:Conn_02x04_Odd_Even
- removed JP1, JP2, JP3: SolderJumper_2_Bridged, Jumper:SolderJumper-2_P1.3mm_Bridged_RoundedPad1.0x1.5mm, symbol Jumper:SolderJumper_2_Bridged
- removed Q1: MMBT2222A, Package_TO_SOT_SMD:SOT-23, symbol Transistor_BJT:PN2222A
- removed R1: 1k, Resistor_SMD:R_0603_1608Metric_Pad0.98x0.95mm_HandSolder, symbol Device:R
- removed R2, R4, R5, R6: 12k, Resistor_SMD:R_0603_1608Metric_Pad0.98x0.95mm_HandSolder, symbol Device:R
- removed R7: 100R, Resistor_SMD:R_0603_1608Metric_Pad0.98x0.95mm_HandSolder, symbol Device:R
- removed U2: LM75B, Package_SO:SOIC-8_3.9x4.9mm_P1.27mm, symbol Sensor_Temperature:LM75B
- removed U3: 74LVC3G17, Package_SO:VSSOP-8_2.3x2mm_P0.5mm, symbol 74xGxx:74LVC3G17
- added DS1: OLED-128O064D, Display:OLED-128O064D, symbol Display_Graphic:OLED-128O064D
- added U4: DS18B20U, Package_SO:MSOP-8_3x3mm_P0.65mm, symbol Sensor_Temperature:DS18B20U
Connections:
- net +3V3: now also JP4.1 (A); no longer JP5.2 (B)
- net +5V: now also JP5.2 (B); no longer JP4.1 (A)
- net GND: now also U4.4 (GND)
- net PSU_SDA: no longer R13.2
- net VCC: now also R3.2, U4.8 (V_{DD}); no longer R3.1
- new net: DS1.1 (GND), DS1.30 (GND)
- new net DQ: R13.2, R3.1, U4.1 (DQ)
- no-connect marks 1 -> 0
Other:
- note added: "Ambient temperature sensing"
- note added: "Display"
- note removed: "Display interface"
- note removed: "I2C sniffer"
- note removed: "Saleae interface"
- note removed: "Temperature sensing"
- note removed: "Voltage sensing"
- moved on the sheet: C13, C14, C3, C4, C5, C6, C7, C8, C9, D2, D3, J3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
